Commit message: optimize build map

File: src/simulated_chassis/urdf/three_wheel_chassis.xacro (robot description, xacro)
@@ -14,5 +14,7 @@
       <origin xyz="0 0 0" rpy="0 0 0" />
       <mass value="60.0" />
-      <inertia ixx="0.5" ixy="0.0" ixz="0.0" iyy="0.5" iyz="0.0" izz="0.8" />
+      <inertia ixx="1.0" ixy="0.0" ixz="0.0"
+         iyy="2.0" iyz="0.0"
+         izz="2.6" />
     </inertial>
     <visual>
@@ -103,6 +105,8 @@
     <inertial>
       <origin xyz="0 0 0" rpy="0 0 0" />
-      <mass value="1.0" />
-      <inertia ixx="0.015" ixy="0.0" ixz="0.0" iyy="0.015" iyz="0.0" izz="0.02" />
+        <mass value="3.0" />
+        <inertia ixx="0.0091" ixy="0.0" ixz="0.0"
+                iyy="0.0091" iyz="0.0"
+                izz="0.015" />
     </inertial>
     <visual>
@@ -133,6 +137,8 @@
     <inertial>
       <origin xyz="0 0 0" rpy="0 0 0" />
-      <mass value="0.5" />
-      <inertia ixx="0.001" ixy="0.0" ixz="0.0" iyy="0.001" iyz="0.0" izz="0.001" />
+        <mass value="3.0" />
+        <inertia ixx="0.0091" ixy="0.0" ixz="0.0"
+                iyy="0.0091" iyz="0.0"
+                izz="0.015" />
     </inertial>
     <visual>
@@ -154,6 +160,8 @@
     <inertial>
       <origin xyz="0 0 0" rpy="0 0 0" />
-      <mass value="1.0" />
-      <inertia ixx="0.015" ixy="0.0" ixz="0.0" iyy="0.015" iyz="0.0" izz="0.02" />
+        <mass value="3.0" />
+        <inertia ixx="0.0091" ixy="0.0" ixz="0.0"
+                iyy="0.0091" iyz="0.0"
+                izz="0.015" />
     </inertial>
     <visual>
@@ -184,6 +192,8 @@
     <inertial>
       <origin xyz="0 0 0" rpy="0 0 0" />
-      <mass value="0.5" />
-      <inertia ixx="0.001" ixy="0.0" ixz="0.0" iyy="0.001" iyz="0.0" izz="0.001" />
+        <mass value="3.0" />
+        <inertia ixx="0.0091" ixy="0.0" ixz="0.0"
+                iyy="0.0091" iyz="0.0"
+                izz="0.015" />
     </inertial>
     <visual>
@@ -205,6 +215,8 @@
     <inertial>
       <origin xyz="0 0 0" rpy="0 0 0" />
-      <mass value="1.0" />
-      <inertia ixx="0.015" ixy="0.0" ixz="0.0" iyy="0.015" iyz="0.0" izz="0.02" />
+        <mass value="3.0" />
+        <inertia ixx="0.0091" ixy="0.0" ixz="0.0"
+                iyy="0.0091" iyz="0.0"
+                izz="0.015" />
     </inertial>
     <visual>
@@ -370,3 +382,34 @@
     </sensor>
   </gazebo>
+  <!-- 在 robot 标签的末尾，为每个车轮的 link 指定摩擦参数 -->
+  <gazebo reference="wheel_front_wheel_link">
+    <surface>
+      <friction>
+        <ode>
+          <mu>0.8</mu>
+          <mu2>0.6</mu2>
+        </ode>
+      </friction>
+    </surface>
+  </gazebo>
+  <gazebo reference="wheel_left_wheel_link">
+    <surface>
+      <friction>
+        <ode>
+          <mu>0.8</mu>
+          <mu2>0.6</mu2>
+        </ode>
+      </friction>
+    </surface>
+  </gazebo>
+  <gazebo reference="wheel_right_wheel_link">
+    <surface>
+      <friction>
+        <ode>
+          <mu>0.8</mu>
+          <mu2>0.6</mu2>
+        </ode>
+      </friction>
+    </surface>
+  </gazebo>
 </robot>

Commit message: lua optimize

File: src/simulated_chassis/urdf/three_wheel_chassis.xacro (robot description, xacro)
@@ -82,6 +82,6 @@
     <inertial>
       <origin xyz="0 0 0" rpy="0 0 0" />
-      <mass value="0.5" />
-      <inertia ixx="0.001" ixy="0.0" ixz="0.0" iyy="0.001" iyz="0.0" izz="0.001" />
+      <mass value="1.5" />
+      <inertia ixx="0.0045" ixy="0.0" ixz="0.0" iyy="0.0045" iyz="0.0" izz="0.0075" />
     </inertial>
     <visual>
@@ -116,5 +116,5 @@
       </geometry>
       <material name="orange_wheel">
-        <color rgba="1.0 0.5 0.0 1.0" />
+        <color rgba="1.0 0.35 0.0 1.0" />
       </material>
     </visual>
@@ -137,8 +137,8 @@
     <inertial>
       <origin xyz="0 0 0" rpy="0 0 0" />
-        <mass value="3.0" />
-        <inertia ixx="0.0091" ixy="0.0" ixz="0.0"
-                iyy="0.0091" iyz="0.0"
-                izz="0.015" />
+        <mass value="1.5" />
+        <inertia ixx="0.0045" ixy="0.0" ixz="0.0"
+                iyy="0.0045" iyz="0.0"
+                izz="0.0075" />
     </inertial>
     <visual>
@@ -171,5 +171,5 @@
       </geometry>
       <material name="orange_wheel">
-        <color rgba="1.0 0.5 0.0 1.0" />
+        <color rgba="1.0 0.35 0.0 1.0" />
       </material>
     </visual>
@@ -192,8 +192,8 @@
     <inertial>
       <origin xyz="0 0 0" rpy="0 0 0" />
-        <mass value="3.0" />
-        <inertia ixx="0.0091" ixy="0.0" ixz="0.0"
-                iyy="0.0091" iyz="0.0"
-                izz="0.015" />
+        <mass value="1.5" />
+        <inertia ixx="0.0045" ixy="0.0" ixz="0.0"
+                iyy="0.0045" iyz="0.0"
+                izz="0.0075" />
     </inertial>
     <visual>
@@ -226,5 +226,5 @@
       </geometry>
       <material name="orange_wheel">
-        <color rgba="1.0 0.5 0.0 1.0" />
+        <color rgba="1.0 0.35 0.0 1.0" />
       </material>
     </visual>
@@ -338,5 +338,5 @@
             <noise type="gaussian">
               <mean>0</mean>
-              <stddev>0.005</stddev>
+              <stddev>0.001</stddev>
             </noise>
           </z>
@@ -346,7 +346,8 @@
   </gazebo>
   <!-- ==================== 3D Lidar ==================== -->
+  <!-- 模拟真实32线雷达：底部密集（地面约束）上部稀疏 -->
+  <!-- 角度分布：±5°内12条线(37.5%)，±5°~±15°16条线(50%)，±15°~±20°4条线(12.5%) -->
   <gazebo reference="lidar_link">
     <sensor name="mid360_sensor" type="gpu_lidar">
-      <!-- <enable>true</enable> -->
       <always_on>true</always_on>
       <update_rate>20</update_rate>
@@ -365,11 +366,11 @@
           <vertical>
             <samples>32</samples>
-            <min_angle>-0.349</min_angle>   <!-- ±20° 视野更大 -->
-            <max_angle>0.349</max_angle>
+            <min_angle>-0.1745</min_angle>   <!-- ±10° 点云集中 -->
+            <max_angle>0.1745</max_angle>
           </vertical>
         </scan>
         <range>
           <min>0.2</min>
-          <max>45.0</max>
+          <max>30.0</max>
           <resolution>0.01</resolution>
         </range>

Commit message: 双3D雷达,还在调整中

File: src/simulated_chassis/urdf/three_wheel_chassis.xacro (robot description, xacro)
@@ -56,6 +56,8 @@
     <origin xyz="0 0 0" rpy="0 0 0" />
   </joint>
-  <!-- ==================== 3D Lidar ==================== -->
-  <link name="lidar_link">
+  <!-- ==================== 3D Lidar 双雷达（前+后，Mid-360 仿真） ==================== -->
+  <!-- 前雷达：底盘前部中央，前倾10°(rpy.pitch=+0.1745，顶部向前) -->
+  <!--   → 下沿射线斜向前下方(-7°+10°倾斜 ≈ 等效-17°)，覆盖机器人正前方地面 -->
+  <link name="front_lidar_link">
     <inertial>
       <origin xyz="0 0 0" rpy="0 0 0" />
@@ -63,18 +65,60 @@
       <inertia ixx="0.001" ixy="0.0" ixz="0.0" iyy="0.001" iyz="0.0" izz="0.001" />
     </inertial>
-    <visual>
-      <origin xyz="0 0 0" rpy="0 0 0" />
-      <geometry>
-        <cylinder radius="0.04" length="0.03" />
-      </geometry>
-      <material name="cinnabar">
-        <color rgba="0.906 0.337 0.196 1.0" />
-      </material>
-    </visual>
-  </link>
-  <joint name="lidar_joint" type="fixed">
+    <!-- 半球穹顶雷达外形：底座圆柱 + 球体(下半埋入底座，只露上半球)，仿 Mid-360 -->
+    <visual>
+      <origin xyz="0 0 0.02" rpy="0 0 0" />
+      <geometry>
+        <cylinder radius="0.04" length="0.04" />
+      </geometry>
+      <material name="lidar_base">
+        <color rgba="0.12 0.12 0.12 1.0" />
+      </material>
+    </visual>
+    <visual>
+      <origin xyz="0 0 0.04" rpy="0 0 0" />
+      <geometry>
+        <sphere radius="0.04" />
+      </geometry>
+      <material name="lidar_dome">
+        <color rgba="0.22 0.22 0.22 1.0" />
+      </material>
+    </visual>
+  </link>
+  <joint name="front_lidar_joint" type="fixed">
     <parent link="base_link" />
-    <child link="lidar_link" />
-    <origin xyz="0 0 0.24" rpy="0 0 0" />
+    <child link="front_lidar_link" />
+    <origin xyz="0.25 0 0.10" rpy="0 0.0873 0" />
+  </joint>
+  <!-- 后雷达：底盘后部中央，朝后(yaw=π)+后倾10° → 覆盖机器人正后方地面 -->
+  <link name="rear_lidar_link">
+    <inertial>
+      <origin xyz="0 0 0" rpy="0 0 0" />
+      <mass value="0.2" />
+      <inertia ixx="0.001" ixy="0.0" ixz="0.0" iyy="0.001" iyz="0.0" izz="0.001" />
+    </inertial>
+    <!-- 半球穹顶雷达外形：底座圆柱 + 球体(下半埋入底座，只露上半球)，仿 Mid-360 -->
+    <visual>
+      <origin xyz="0 0 0.02" rpy="0 0 0" />
+      <geometry>
+        <cylinder radius="0.04" length="0.04" />
+      </geometry>
+      <material name="lidar_base">
+        <color rgba="0.12 0.12 0.12 1.0" />
+      </material>
+    </visual>
+    <visual>
+      <origin xyz="0 0 0.04" rpy="0 0 0" />
+      <geometry>
+        <sphere radius="0.04" />
+      </geometry>
+      <material name="lidar_dome">
+        <color rgba="0.22 0.22 0.22 1.0" />
+      </material>
+    </visual>
+  </link>
+  <joint name="rear_lidar_joint" type="fixed">
+    <parent link="base_link" />
+    <child link="rear_lidar_link" />
+    <origin xyz="-0.25 0 0.10" rpy="0 0.0873 3.1416" />
   </joint>
   <!-- ==================== Front Steering Module ==================== -->
@@ -347,34 +391,32 @@
     </sensor>
   </gazebo>
-  <!-- ==================== 3D Lidar ==================== -->
-  <!-- 模拟真实32线雷达：底部密集（地面约束）上部稀疏 -->
-  <!-- 角度分布：±5°内12条线(37.5%)，±5°~±15°16条线(50%)，±15°~±20°4条线(12.5%) -->
-  <gazebo reference="lidar_link">
-    <sensor name="mid360_sensor" type="gpu_lidar">
-      <!-- <enable>true</enable> -->
+  <!-- ==================== 双 3D Lidar Sensor (Mid-360 仿真) ==================== -->
+  <!-- 垂直视场非对称：下沿 -7°(真实Mid-360) / 上沿 +32°。前后两个传感器配置完全一致。 -->
+  <!-- 前雷达 -->
+  <gazebo reference="front_lidar_link">
+    <sensor name="front_lidar_sensor" type="gpu_lidar">
       <always_on>true</always_on>
       <update_rate>15</update_rate>
       <visualize>true</visualize>
-      <topic>/lidar/point_cloud</topic>
-      <ignition_frame_id>lidar_link</ignition_frame_id>
+      <topic>/front_lidar/point_cloud</topic>
+      <ignition_frame_id>front_lidar_link</ignition_frame_id>
       <lidar>
-        <frame_id>lidar_link</frame_id>
+        <frame_id>front_lidar_link</frame_id>
         <scan>
           <horizontal>
-            <samples>360</samples>
+            <samples>270</samples>
             <resolution>1</resolution>
-            <min_angle>-3.1415926</min_angle>
-            <max_angle>3.1415926</max_angle>
+            <min_angle>-2.3562</min_angle>
+            <max_angle>2.3562</max_angle>
           </horizontal>
-          <!-- ===== 稳定版(v1.0.0-nav-stable)雷达配置，整段覆盖用于对比 ===== -->
           <vertical>
             <samples>32</samples>
-            <min_angle>-0.3490</min_angle>
-            <max_angle>0.3490</max_angle>
+            <min_angle>-0.2618</min_angle>
+            <max_angle>0.349</max_angle>
           </vertical>
         </scan>
         <range>
           <min>0.2</min>
-          <max>45.0</max>
+          <max>30.0</max>
           <resolution>0.01</resolution>
         </range>
@@ -382,8 +424,47 @@
           <type>gaussian</type>
           <mean>0.0</mean>
-          <!-- <stddev>0.182</stddev> -->
           <bias_mean>0.0</bias_mean>
           <bias_stddev>0.005</bias_stddev>
           <precision>0.01</precision>
+          <stddev>0.010</stddev>
+        </noise>
+      </lidar>
+    </sensor>
+  </gazebo>
+  <!-- 后雷达 -->
+  <gazebo reference="rear_lidar_link">
+    <sensor name="rear_lidar_sensor" type="gpu_lidar">
+      <always_on>true</always_on>
+      <update_rate>15</update_rate>
+      <visualize>true</visualize>
+      <topic>/rear_lidar/point_cloud</topic>
+      <ignition_frame_id>rear_lidar_link</ignition_frame_id>
+      <lidar>
+        <frame_id>rear_lidar_link</frame_id>
+        <scan>
+          <horizontal>
+            <samples>270</samples>
+            <resolution>1</resolution>
+            <min_angle>-2.3562</min_angle>
+            <max_angle>2.3562</max_angle>
+          </horizontal>
+          <vertical>
+            <samples>32</samples>
+            <min_angle>-0.2618</min_angle>
+            <max_angle>0.349</max_angle>
+          </vertical>
+        </scan>
+        <range>
+          <min>0.2</min>
+          <max>30.0</max>
+          <resolution>0.01</resolution>
+        </range>
+        <noise>
+          <type>gaussian</type>
+          <mean>0.0</mean>
+          <bias_mean>0.0</bias_mean>
+          <bias_stddev>0.005</bias_stddev>
+          <precision>0.01</precision>
+          <stddev>0.010</stddev>
         </noise>
       </lidar>

Commit message: optime angle

File: src/simulated_chassis/urdf/three_wheel_chassis.xacro (robot description, xacro)
@@ -144,5 +144,5 @@
     <origin xyz="0.3 0.0 -0.05" rpy="0 0 0" />
     <axis xyz="0 0 1" />
-    <limit lower="-3.14159" upper="3.14159" effort="10.0" velocity="5.0" />
+    <limit lower="-1.5708" upper="1.5708" effort="10.0" velocity="5.0" />
   </joint>
   <link name="wheel_front_wheel_link">
@@ -199,5 +199,5 @@
     <origin xyz="-0.15 0.26 -0.05" rpy="0 0 0" />
     <axis xyz="0 0 1" />
-    <limit lower="-3.14159" upper="3.14159" effort="10.0" velocity="5.0" />
+    <limit lower="-1.5708" upper="1.5708" effort="10.0" velocity="5.0" />
   </joint>
   <link name="wheel_left_wheel_link">
@@ -254,5 +254,5 @@
     <origin xyz="-0.15 -0.26 -0.05" rpy="0 0 0" />
     <axis xyz="0 0 1" />
-    <limit lower="-3.14159" upper="3.14159" effort="10.0" velocity="5.0" />
+    <limit lower="-1.5708" upper="1.5708" effort="10.0" velocity="5.0" />
   </joint>
   <link name="wheel_right_wheel_link">

Commit message: 雷达贴边低装+点云地面滤除，放宽定位重启健康检查超时
- xacro: 底盘加大至0.8x0.6并对齐惯量，双雷达外移至前后边缘(±0.36外沿对齐)，
  支架从11cm降到1cm（雷达座z=0.10，离地0.25m）
- 新增 pointcloud_ground_filter 节点：base_footprint系高度带裁剪滤地面回波，
  slam/localization launch 重映射至 /points2*_filtered，消除2D地图灰点与z漂移
- agv_bridge_v2: get_trajectory_states 健康检查 60s→150s，
  避免大地图加载期定位进程被误杀（导致建图保存失败）
- 三舵轮控制器/导航参数/rviz 调整，新增 cancel_nav.py 工具，忽略 serverProjects/

File: src/simulated_chassis/urdf/three_wheel_chassis.xacro (robot description, xacro)
@@ -14,12 +14,13 @@
       <origin xyz="0 0 0" rpy="0 0 0" />
       <mass value="60.0" />
-      <inertia ixx="1.0" ixy="0.0" ixz="0.0"
-         iyy="2.0" iyz="0.0"
-         izz="2.6" />
-    </inertial>
-    <visual>
-      <origin xyz="0 0 0" rpy="0 0 0" />
-      <geometry>
-        <box size="0.6 0.4 0.18" />
+      <!-- 惯量按箱体 0.8 x 0.6 x 0.18 公式计算（Ixx=m/12*(y²+z²) 等） -->
+      <inertia ixx="1.96" ixy="0.0" ixz="0.0"
+         iyy="3.36" iyz="0.0"
+         izz="5.0" />
+    </inertial>
+    <visual>
+      <origin xyz="0 0 0" rpy="0 0 0" />
+      <geometry>
+        <box size="0.8 0.6 0.18" />
       </geometry>
       <material name="green">
@@ -30,7 +31,22 @@
       <origin xyz="0 0 0" rpy="0 0 0" />
       <geometry>
-        <box size="0.6 0.4 0.18" />
+        <box size="0.8 0.6 0.18" />
       </geometry>
     </collision>
+    <!-- 雷达安装垫柱（高1cm：底盘顶面 z=0.09 → 雷达座 z=0.10），位置随雷达外移至前后边缘 -->
+    <visual>
+      <origin xyz="0.36 0 0.095" rpy="0 0 0" />
+      <geometry>
+        <cylinder radius="0.025" length="0.01" />
+      </geometry>
+      <material name="grey" />
+    </visual>
+    <visual>
+      <origin xyz="-0.36 0 0.095" rpy="0 0 0" />
+      <geometry>
+        <cylinder radius="0.025" length="0.01" />
+      </geometry>
+      <material name="grey" />
+    </visual>
   </link>
   <!-- ==================== IMU ==================== -->
@@ -57,6 +73,9 @@
   </joint>
   <!-- ==================== 3D Lidar 双雷达（前+后，Mid-360 仿真） ==================== -->
-  <!-- 前雷达：底盘前部中央，前倾10°(rpy.pitch=+0.1745，顶部向前) -->
-  <!--   → 下沿射线斜向前下方(-7°+10°倾斜 ≈ 等效-17°)，覆盖机器人正前方地面 -->
+  <!-- 雷达经1cm垫柱安装在底盘顶面（雷达座 z=0.10，世界高度0.25），并外移至前后边缘：
+       底座半径0.04，中心取±0.36 使外沿与底盘边缘(±0.4)对齐，
+       前后向俯角射线出射即越过底盘边缘；侧向>约2°的俯角射线会打在自家底盘上，
+       机身两侧近处存在小范围盲区 -->
+  <!-- 前雷达：底盘前边缘，前倾5°(rpy.pitch=+0.0873，顶部向前) -->
   <link name="front_lidar_link">
     <inertial>
@@ -88,7 +107,7 @@
     <parent link="base_link" />
     <child link="front_lidar_link" />
-    <origin xyz="0.25 0 0.10" rpy="0 0.0873 0" />
-  </joint>
-  <!-- 后雷达：底盘后部中央，朝后(yaw=π)+后倾10° → 覆盖机器人正后方地面 -->
+    <origin xyz="0.36 0 0.10" rpy="0 0.0873 0" />
+  </joint>
+  <!-- 后雷达：底盘后边缘，朝后(yaw=π)+后倾5° → 覆盖机器人正后方 -->
   <link name="rear_lidar_link">
     <inertial>
@@ -120,5 +139,5 @@
     <parent link="base_link" />
     <child link="rear_lidar_link" />
-    <origin xyz="-0.25 0 0.10" rpy="0 0.0873 3.1416" />
+    <origin xyz="-0.36 0 0.10" rpy="0 0.0873 3.1416" />
   </joint>
   <!-- ==================== Front Steering Module ==================== -->
@@ -197,5 +216,5 @@
     <parent link="base_link" />
     <child link="wheel_left_steering_link" />
-    <origin xyz="-0.15 0.26 -0.05" rpy="0 0 0" />
+    <origin xyz="-0.15 0.20 -0.05" rpy="0 0 0" />
     <axis xyz="0 0 1" />
     <limit lower="-1.5708" upper="1.5708" effort="10.0" velocity="5.0" />
@@ -252,5 +271,5 @@
     <parent link="base_link" />
     <child link="wheel_right_steering_link" />
-    <origin xyz="-0.15 -0.26 -0.05" rpy="0 0 0" />
+    <origin xyz="-0.15 -0.20 -0.05" rpy="0 0 0" />
     <axis xyz="0 0 1" />
     <limit lower="-1.5708" upper="1.5708" effort="10.0" velocity="5.0" />
