Commit message: build map and navigation

File: src/simulated_chassis/urdf/three_wheel_chassis copy.xacro (robot description, xacro)
@@ -2,4 +2,5 @@
 <robot xmlns:xacro="http://www.ros.org/wiki/xacro" name="three_wheel_agv">
   <!-- ==================== Base Footprint ==================== -->
+  <!-- 机器人在地面的投影点，用于导航和 TF 树 -->
   <link name="base_footprint">
   </link>
@@ -7,5 +8,6 @@
     <parent link="base_footprint"/>
     <child link="base_link"/>
-    <origin xyz="0 0 0.15" rpy="0 0 0"/>
+    <!-- base_link 中心高度 0.175，所以 footprint 在 base_link 下方 0.175 -->
+    <origin xyz="0 0 0.175" rpy="0 0 0"/>
   </joint>
   <!-- ==================== Base Link ==================== -->
@@ -13,4 +15,5 @@
     <inertial>
       <origin xyz="0 0 0" rpy="0 0 0"/>
+      <!-- 质心在原点 -->
       <mass value="60.0"/>
       <inertia ixx="0.5" ixy="0.0" ixz="0.0" iyy="0.5" iyz="0.0" izz="0.8"/>
@@ -18,6 +21,7 @@
     <visual>
       <origin xyz="0 0 0" rpy="0 0 0"/>
-      <geometry>
-        <box size="0.6 0.4 0.18"/>
+      <!-- 视觉在原点 -->
+      <geometry>
+        <box size="0.6 0.4 0.15"/>
       </geometry>
       <material name="green">
@@ -27,6 +31,7 @@
     <collision>
       <origin xyz="0 0 0" rpy="0 0 0"/>
-      <geometry>
-        <box size="0.6 0.4 0.18"/>
+      <!-- 碰撞在原点 -->
+      <geometry>
+        <box size="0.6 0.4 0.15"/>
       </geometry>
     </collision>
@@ -46,4 +51,5 @@
       <material name="purple">
         <color rgba="0.8 0.0 0.8 1.0"/>
+        <!-- 紫色 -->
       </material>
     </visual>
@@ -54,5 +60,5 @@
     <origin xyz="0 0 0" rpy="0 0 0"/>
   </joint>
-  <!-- ==================== 3D Lidar ==================== -->
+  <!-- ==================== 3D Lidar (Mid360 style) ==================== -->
   <link name="lidar_link">
     <inertial>
@@ -74,5 +80,5 @@
     <parent link="base_link"/>
     <child link="lidar_link"/>
-    <origin xyz="0 0 0.24" rpy="0 0 0"/>
+    <origin xyz="0 0 0.32" rpy="0 0 0"/>
   </joint>
   <!-- ==================== Front Steering Module ==================== -->
@@ -96,6 +102,7 @@
     <parent link="base_link"/>
     <child link="wheel_front_steering_link"/>
-    <origin xyz="0.3 0.0 -0.05" rpy="0 0 0"/>
+    <origin xyz="0.3 0.0 0.1" rpy="0 0 0"/>
     <axis xyz="0 0 1"/>
+    <!-- 360° 转向支持 -->
     <limit lower="-3.14159" upper="3.14159" effort="10.0" velocity="5.0"/>
   </joint>
@@ -113,4 +120,5 @@
       <material name="orange_wheel">
         <color rgba="1.0 0.5 0.0 1.0"/>
+        <!-- 橙色 -->
       </material>
     </visual>
@@ -147,5 +155,5 @@
     <parent link="base_link"/>
     <child link="wheel_left_steering_link"/>
-    <origin xyz="-0.15 0.26 -0.05" rpy="0 0 0"/>
+    <origin xyz="-0.15 0.26 0.1" rpy="0 0 0"/>
     <axis xyz="0 0 1"/>
     <limit lower="-3.14159" upper="3.14159" effort="10.0" velocity="5.0"/>
@@ -164,4 +172,5 @@
       <material name="orange_wheel">
         <color rgba="1.0 0.5 0.0 1.0"/>
+        <!-- 橙色 -->
       </material>
     </visual>
@@ -198,5 +207,5 @@
     <parent link="base_link"/>
     <child link="wheel_right_steering_link"/>
-    <origin xyz="-0.15 -0.26 -0.05" rpy="0 0 0"/>
+    <origin xyz="-0.15 -0.26 0.1" rpy="0 0 0"/>
     <axis xyz="0 0 1"/>
     <limit lower="-3.14159" upper="3.14159" effort="10.0" velocity="5.0"/>
@@ -215,4 +224,5 @@
       <material name="orange_wheel">
         <color rgba="1.0 0.5 0.0 1.0"/>
+        <!-- 橙色 -->
       </material>
     </visual>
@@ -273,10 +283,14 @@
       <robot_param>robot_description</robot_param>
       <robot_param_node>robot_state_publisher</robot_param_node>
+      <!-- <robot_base_name>base_footprint</robot_base_name> -->
     </plugin>
     <plugin filename="ignition-gazebo-sensors-system" name="ignition::gazebo::systems::Sensors">
     </plugin>
     <plugin name="ignition::gazebo::systems::Imu" filename="ignition-gazebo-imu-system"></plugin>
+    <!-- <plugin name='ignition::gazebo::systems::Physics' filename='ignition-gazebo-physics-system'></plugin>
+    <plugin name='ignition::gazebo::systems::UserCommands' filename='ignition-gazebo-user-commands-system'></plugin>
+    <plugin name='ignition::gazebo::systems::SceneBroadcaster' filename='ignition-gazebo-scene-broadcaster-system'></plugin> -->
   </gazebo>
-  <!-- ==================== IMU Sensor ==================== -->
+  <!-- ==================== IMU Sensor (Edifice Compatible) ==================== -->
   <gazebo reference="imu_link">
     <sensor name="imu_sensor" type="imu">
@@ -331,6 +345,5 @@
     </sensor>
   </gazebo>
-  <!-- ==================== 3D Lidar ==================== -->
- <gazebo reference="lidar_link">
+  <gazebo reference="lidar_link">
     <sensor name="mid360_sensor" type="gpu_lidar">
       <enable>true</enable>
