Commit message: 三舵轮3D链路大修：tracked_pose重锚定根治TF拆分抖动 + 控制器位置差分里程计
- 抖动根治：carto停发TF改发/tracked_pose(publish_to_tf=false)，新增
  tracked_pose_tf_node同一时间戳重锚定发map->odom，消除外推值与旧时刻
  odom锚定的双重计数（前进-回退锯齿）与关外推后的步进卡顿
- 控制器：里程计改轮位置差分（diff_drive同款，回绕折回(−π,π]免疫），
  无门控纯测量；舵关节effort 10→100根治静摩擦转向死锁；creep=0
  排除刮擦幻影里程；位置控制增益0.3
- 雷达：3D版垂直FOV -25°→-10°（原俯角射线自打底盘前边缘，眼前幻影
  障碍致导航减速），16线/360采样/量程0.3-30对齐zioneer验证版
- launch默认全链路切回3D（xacro/bridge/建图/定位/导航/离线）
- zioneer：脚轮预紧方向反转修复动力轮悬空空转、雷达降高1cm垫柱、
  open_loop=false实测里程计、cmd_vel_timeout 1.5防断流刹车抖动
- bridge：save_map响应超时15→40s+回退补导出前等3s+map_saver等图
  10→30s（CPU饱和时误杀慢速保存的根因）
- 日志降噪：rosbridge提WARN级、LocalizationMonitor TF树转储转DEBUG
- occupancy grid发布1Hz→0.2Hz（websocket带宽省80%）
- 本提交同时恢复被加密软件批量还原到旧快照的以上全部代码

File: src/simulated_chassis/urdf/three_wheel_chassis_3d.xacro (robot description, xacro)
@@ -1,4 +1,8 @@
 <?xml version="1.0"?>
 <robot xmlns:xacro="http://www.ros.org/wiki/xacro" name="three_wheel_agv">
+  <!-- 全局材质定义：垫柱/转向节引用的 grey 之前未定义，触发 urdf_parser 警告 -->
+  <material name="grey">
+    <color rgba="0.5 0.5 0.5 1.0" />
+  </material>
   <!-- ==================== Base Footprint ==================== -->
   <link name="base_footprint">
@@ -161,5 +165,5 @@
     <origin xyz="0.3 0.0 -0.05" rpy="0 0 0" />
     <axis xyz="0 0 1" />
-    <limit lower="-1.5708" upper="1.5708" effort="10.0" velocity="5.0" />
+    <limit lower="-1.5708" upper="1.5708" effort="100.0" velocity="5.0" />
   </joint>
   <link name="wheel_front_wheel_link">
@@ -212,5 +216,5 @@
     <origin xyz="-0.15 0.20 -0.05" rpy="0 0 0" />
     <axis xyz="0 0 1" />
-    <limit lower="-1.5708" upper="1.5708" effort="10.0" velocity="5.0" />
+    <limit lower="-1.5708" upper="1.5708" effort="100.0" velocity="5.0" />
   </joint>
   <link name="wheel_left_wheel_link">
@@ -263,5 +267,5 @@
     <origin xyz="-0.15 -0.20 -0.05" rpy="0 0 0" />
     <axis xyz="0 0 1" />
-    <limit lower="-1.5708" upper="1.5708" effort="10.0" velocity="5.0" />
+    <limit lower="-1.5708" upper="1.5708" effort="100.0" velocity="5.0" />
   </joint>
   <link name="wheel_right_wheel_link">
@@ -439,18 +443,21 @@
         <scan>
           <horizontal>
-            <samples>270</samples>
+            <samples>360</samples>
             <resolution>1</resolution>
-            <min_angle>-2.3562</min_angle>
-            <max_angle>2.3562</max_angle>
+            <min_angle>-2.35619</min_angle>
+            <max_angle>2.35619</max_angle>
           </horizontal>
+          <!-- 对齐 zioneer 差速版：下沿 -10°。原 -25° 俯角射线会打在自己底盘前边缘
+               （雷达在边缘内 4cm、甲板仅低 1cm，≥14° 俯角即自打），眼前出现幻影障碍
+               导致导航减速。-10° 时打中甲板需 ≥27°，几何上不可能自打。 -->
           <vertical>
-            <samples>32</samples>
-            <min_angle>-0.4363</min_angle>            <!-- -25° -->
-            <max_angle>0.3491</max_angle>            <!-- +20° -->
+            <samples>16</samples>
+            <min_angle>-0.1745</min_angle>            <!-- -10° -->
+            <max_angle>0.349</max_angle>              <!-- +20° -->
           </vertical>
         </scan>
         <range>
-          <min>0.55</min>
-          <max>45.0</max>
+          <min>0.3</min>
+          <max>30.0</max>
           <resolution>0.01</resolution>
         </range>
@@ -459,7 +466,7 @@
           <mean>0.0</mean>
           <bias_mean>0.0</bias_mean>
-          <bias_stddev>0.005</bias_stddev>
+          <bias_stddev>0.0005</bias_stddev>
           <precision>0.01</precision>
-          <stddev>0.010</stddev>
+          <stddev>0.002</stddev>
         </noise>
       </lidar>
@@ -478,18 +485,19 @@
         <scan>
           <horizontal>
-            <samples>270</samples>
+            <samples>360</samples>
             <resolution>1</resolution>
-            <min_angle>-2.3562</min_angle>
-            <max_angle>2.3562</max_angle>
+            <min_angle>-2.35619</min_angle>
+            <max_angle>2.35619</max_angle>
           </horizontal>
+          <!-- 对齐 zioneer 差速版：下沿 -10°，杜绝俯角射线自打底盘边缘 -->
           <vertical>
-            <samples>32</samples>
-            <min_angle>-0.4363</min_angle>            <!-- -25° -->
-            <max_angle>0.3491</max_angle>            <!-- +20° -->
+            <samples>16</samples>
+            <min_angle>-0.1745</min_angle>            <!-- -10° -->
+            <max_angle>0.349</max_angle>              <!-- +20° -->
           </vertical>
         </scan>
         <range>
-          <min>0.55</min>
-          <max>45.0</max>
+          <min>0.3</min>
+          <max>30.0</max>
           <resolution>0.01</resolution>
         </range>
@@ -498,7 +506,7 @@
           <mean>0.0</mean>
           <bias_mean>0.0</bias_mean>
-          <bias_stddev>0.005</bias_stddev>
+          <bias_stddev>0.0005</bias_stddev>
           <precision>0.01</precision>
-          <stddev>0.010</stddev>
+          <stddev>0.002</stddev>
         </noise>
       </lidar>

File: src/zioneer_robot/urdf/diff/diff_base.xacro (robot description, xacro)
@@ -28,4 +28,21 @@
         </inertial>
     </link>
+    <!-- 雷达安装垫柱（高1cm：底盘顶面 z=0.06 -> 雷达座 z=0.07），位置随雷达外移至前后边缘 -->
+    <visual>
+        <origin xyz="0.28 0 0.065" rpy="0 0 0" />
+        <geometry>
+            <cylinder radius="0.025" length="0.01" />
+        </geometry>
+        <material name="mount_pad">
+            <color rgba="0.3 0.3 0.3 1.0" />
+        </material>
+    </visual>
+    <visual>
+        <origin xyz="-0.28 0 0.065" rpy="0 0 0" />
+        <geometry>
+            <cylinder radius="0.025" length="0.01" />
+        </geometry>
+        <material name="mount_pad" />
+    </visual>
     <gazebo reference="base_link">
         <material>Gazebo/Orange</material>
@@ -57,5 +74,6 @@
         <parent link="base_link" />
         <child link="front_lidar_link" />
-        <origin xyz="0.28 0 0.20" rpy="0 0 0" />
+        <!-- 1cm 垫柱安装：雷达座 z=0.07（世界高 0.22），不倾斜 -->
+        <origin xyz="0.28 0 0.07" rpy="0 0 0" />
     </joint>
     <!-- ==================== 后3D雷达 (Mid-360 仿真) ==================== -->
@@ -84,5 +102,6 @@
         <parent link="base_link" />
         <child link="rear_lidar_link" />
-        <origin xyz="-0.28 0 0.20" rpy="0 0 3.1416" />
+        <!-- 1cm 垫柱安装：雷达座 z=0.07（世界高 0.22），朝后 yaw=π，不倾斜 -->
+        <origin xyz="-0.28 0 0.07" rpy="0 0 3.1416" />
     </joint>
     <!-- ==================== IMU ==================== -->

File: src/zioneer_robot/urdf/diff/diff_wheels.xacro (robot description, xacro)
@@ -108,8 +108,11 @@
         </joint>
     </xacro:macro>
-    <!-- 四个脚轮：z=-0.1205，底部低于地面0.5mm预紧，防止机器人两点支撑翘起1.1° -->
-    <xacro:caster_wheel prefix="caster_front_right" x="0.24" y="0.14" z="-0.1205" />
-    <xacro:caster_wheel prefix="caster_front_left"  x="0.24" y="-0.14" z="-0.1205" />
-    <xacro:caster_wheel prefix="caster_rear_right"  x="-0.24" y="0.14" z="-0.1205" />
-    <xacro:caster_wheel prefix="caster_rear_left"   x="-0.24" y="-0.14" z="-0.1205" />
+    <!-- 四个防倾垫（fixed 实心圆柱，非滚轮）：底面抬到轮底平面上方 2.5mm，
+         动力轮承重、垫悬空；只有车身倾斜 >0.55°(2.5mm/0.26m) 时垫才触地防翻。
+         注意方向：垫绝不能低于轮底，否则整车压在垫上、动力轮悬空空转
+         （实测 3.33 rad/s 空转零位移、激光无近障，即此因）。 -->
+    <xacro:caster_wheel prefix="caster_front_right" x="0.24" y="0.14" z="-0.1175" />
+    <xacro:caster_wheel prefix="caster_front_left"  x="0.24" y="-0.14" z="-0.1175" />
+    <xacro:caster_wheel prefix="caster_rear_right"  x="-0.24" y="0.14" z="-0.1175" />
+    <xacro:caster_wheel prefix="caster_rear_left"   x="-0.24" y="-0.14" z="-0.1175" />
 </robot>

Commit message: 将机械臂集成到仿真机器人上面，做成复合机器人

File: src/simulated_chassis/urdf/three_wheel_chassis_3d.xacro (robot description, xacro)
@@ -1,546 +1,5 @@
 <?xml version="1.0"?>
 <robot xmlns:xacro="http://www.ros.org/wiki/xacro" name="three_wheel_agv">
-  <!-- 全局材质定义：垫柱/转向节引用的 grey 之前未定义，触发 urdf_parser 警告 -->
-  <material name="grey">
-    <color rgba="0.5 0.5 0.5 1.0" />
-  </material>
-  <!-- ==================== Base Footprint ==================== -->
-  <link name="base_footprint">
-  </link>
-  <joint name="base_footprint_joint" type="fixed">
-    <parent link="base_footprint" />
-    <child link="base_link" />
-    <origin xyz="0 0 0.15" rpy="0 0 0" />
-  </joint>
-  <!-- ==================== Base Link ==================== -->
-  <link name="base_link">
-    <inertial>
-      <origin xyz="0 0 0" rpy="0 0 0" />
-      <mass value="60.0" />
-      <!-- 惯量按箱体 0.8 x 0.6 x 0.18 公式计算（Ixx=m/12*(y²+z²) 等） -->
-      <inertia ixx="1.96" ixy="0.0" ixz="0.0" iyy="3.36" iyz="0.0" izz="5.0" />
-    </inertial>
-    <visual>
-      <origin xyz="0 0 0" rpy="0 0 0" />
-      <geometry>
-        <box size="0.8 0.6 0.18" />
-      </geometry>
-      <material name="green">
-        <color rgba="0.1 0.8 0.1 1.0" />
-      </material>
-    </visual>
-    <collision>
-      <origin xyz="0 0 0" rpy="0 0 0" />
-      <geometry>
-        <box size="0.8 0.6 0.18" />
-      </geometry>
-    </collision>
-    <!-- 雷达安装垫柱（高1cm：底盘顶面 z=0.09 → 雷达座 z=0.10），位置随雷达外移至前后边缘 -->
-    <visual>
-      <origin xyz="0.36 0 0.095" rpy="0 0 0" />
-      <geometry>
-        <cylinder radius="0.025" length="0.01" />
-      </geometry>
-      <material name="grey" />
-    </visual>
-    <visual>
-      <origin xyz="-0.36 0 0.095" rpy="0 0 0" />
-      <geometry>
-        <cylinder radius="0.025" length="0.01" />
-      </geometry>
-      <material name="grey" />
-    </visual>
-  </link>
-  <!-- ==================== IMU ==================== -->
-  <link name="imu_link">
-    <inertial>
-      <origin xyz="0 0 0" rpy="0 0 0" />
-      <mass value="0.01" />
-      <inertia ixx="0.0001" ixy="0.0" ixz="0.0" iyy="0.0001" iyz="0.0" izz="0.0001" />
-    </inertial>
-    <visual>
-      <origin xyz="0 0 0" rpy="0 0 0" />
-      <geometry>
-        <box size="0.04 0.04 0.02" />
-      </geometry>
-      <material name="purple">
-        <color rgba="0.8 0.0 0.8 1.0" />
-      </material>
-    </visual>
-  </link>
-  <joint name="imu_joint" type="fixed">
-    <parent link="base_link" />
-    <child link="imu_link" />
-    <origin xyz="0 0 0" rpy="0 0 0" />
-  </joint>
-  <!-- ==================== 3D Lidar 双雷达（前+后，Mid-360 仿真） ==================== -->
-  <!-- 雷达经1cm垫柱安装在底盘顶面（雷达座 z=0.10，世界高度0.25），并外移至前后边缘：
-       底座半径0.04，中心取±0.36 使外沿与底盘边缘(±0.4)对齐，
-       前后向俯角射线出射即越过底盘边缘；侧向>约2°的俯角射线会打在自家底盘上，
-       机身两侧近处存在小范围盲区 -->
-  <!-- 前雷达：底盘前边缘，前倾5°(rpy.pitch=+0.0873，顶部向前) -->
-  <link name="front_lidar_link">
-    <inertial>
-      <origin xyz="0 0 0" rpy="0 0 0" />
-      <mass value="0.2" />
-      <inertia ixx="0.001" ixy="0.0" ixz="0.0" iyy="0.001" iyz="0.0" izz="0.001" />
-    </inertial>
-    <!-- 半球穹顶雷达外形：底座圆柱 + 球体(下半埋入底座，只露上半球)，仿 Mid-360 -->
-    <visual>
-      <origin xyz="0 0 0.02" rpy="0 0 0" />
-      <geometry>
-        <cylinder radius="0.04" length="0.04" />
-      </geometry>
-      <material name="lidar_base">
-        <color rgba="0.12 0.12 0.12 1.0" />
-      </material>
-    </visual>
-    <visual>
-      <origin xyz="0 0 0.04" rpy="0 0 0" />
-      <geometry>
-        <sphere radius="0.04" />
-      </geometry>
-      <material name="lidar_dome">
-        <color rgba="0.22 0.22 0.22 1.0" />
-      </material>
-    </visual>
-  </link>
-  <joint name="front_lidar_joint" type="fixed">
-    <parent link="base_link" />
-    <child link="front_lidar_link" />
-    <origin xyz="0.36 0 0.10" rpy="0 0 0" />
-  </joint>
-  <!-- 后雷达：底盘后边缘，朝后(yaw=π)+后倾5° → 覆盖机器人正后方 -->
-  <link name="rear_lidar_link">
-    <inertial>
-      <origin xyz="0 0 0" rpy="0 0 0" />
-      <mass value="0.2" />
-      <inertia ixx="0.001" ixy="0.0" ixz="0.0" iyy="0.001" iyz="0.0" izz="0.001" />
-    </inertial>
-    <!-- 半球穹顶雷达外形：底座圆柱 + 球体(下半埋入底座，只露上半球)，仿 Mid-360 -->
-    <visual>
-      <origin xyz="0 0 0.02" rpy="0 0 0" />
-      <geometry>
-        <cylinder radius="0.04" length="0.04" />
-      </geometry>
-      <material name="lidar_base">
-        <color rgba="0.12 0.12 0.12 1.0" />
-      </material>
-    </visual>
-    <visual>
-      <origin xyz="0 0 0.04" rpy="0 0 0" />
-      <geometry>
-        <sphere radius="0.04" />
-      </geometry>
-      <material name="lidar_dome">
-        <color rgba="0.22 0.22 0.22 1.0" />
-      </material>
-    </visual>
-  </link>
-  <joint name="rear_lidar_joint" type="fixed">
-    <parent link="base_link" />
-    <child link="rear_lidar_link" />
-    <origin xyz="-0.36 0 0.10" rpy="0 0 3.1416" />
-  </joint>
-  <!-- ==================== Front Steering Module ==================== -->
-  <link name="wheel_front_steering_link">
-    <inertial>
-      <origin xyz="0 0 0" rpy="0 0 0" />
-      <mass value="1.5" />
-      <inertia ixx="0.0045" ixy="0.0" ixz="0.0" iyy="0.0045" iyz="0.0" izz="0.0075" />
-    </inertial>
-    <visual>
-      <origin xyz="0 0 0" rpy="0 0 0" />
-      <geometry>
-        <cylinder radius="0.03" length="0.06" />
-      </geometry>
-      <material name="grey">
-        <color rgba="0.5 0.5 0.5 1.0" />
-      </material>
-    </visual>
-  </link>
-  <joint name="wheel_front_steering_joint" type="revolute">
-    <parent link="base_link" />
-    <child link="wheel_front_steering_link" />
-    <origin xyz="0.3 0.0 -0.05" rpy="0 0 0" />
-    <axis xyz="0 0 1" />
-    <limit lower="-1.5708" upper="1.5708" effort="100.0" velocity="5.0" />
-  </joint>
-  <link name="wheel_front_wheel_link">
-    <inertial>
-      <origin xyz="0 0 0" rpy="0 0 0" />
-      <mass value="3.0" />
-      <inertia ixx="0.0091" ixy="0.0" ixz="0.0" iyy="0.0091" iyz="0.0" izz="0.015" />
-    </inertial>
-    <visual>
-      <origin xyz="0 0 0" rpy="1.5708 0 0" />
-      <geometry>
-        <cylinder radius="0.1" length="0.08" />
-      </geometry>
-      <material name="orange_wheel">
-        <color rgba="1.0 0.35 0.0 1.0" />
-      </material>
-    </visual>
-    <collision>
-      <origin xyz="0 0 0" rpy="1.5708 0 0" />
-      <geometry>
-        <cylinder radius="0.1" length="0.08" />
-      </geometry>
-    </collision>
-  </link>
-  <joint name="wheel_front_wheel_joint" type="revolute">
-    <parent link="wheel_front_steering_link" />
-    <child link="wheel_front_wheel_link" />
-    <origin xyz="0.0 0.0 0.0" rpy="0 0 0" />
-    <axis xyz="0 1 0" />
-    <limit lower="-1e9" upper="1e9" effort="10.0" velocity="10.0" />
-  </joint>
-  <!-- ==================== Left Steering Module ==================== -->
-  <link name="wheel_left_steering_link">
-    <inertial>
-      <origin xyz="0 0 0" rpy="0 0 0" />
-      <mass value="1.5" />
-      <inertia ixx="0.0045" ixy="0.0" ixz="0.0" iyy="0.0045" iyz="0.0" izz="0.0075" />
-    </inertial>
-    <visual>
-      <origin xyz="0 0 0" rpy="0 0 0" />
-      <geometry>
-        <cylinder radius="0.03" length="0.06" />
-      </geometry>
-      <material name="grey" />
-    </visual>
-  </link>
-  <joint name="wheel_left_steering_joint" type="revolute">
-    <parent link="base_link" />
-    <child link="wheel_left_steering_link" />
-    <origin xyz="-0.15 0.20 -0.05" rpy="0 0 0" />
-    <axis xyz="0 0 1" />
-    <limit lower="-1.5708" upper="1.5708" effort="100.0" velocity="5.0" />
-  </joint>
-  <link name="wheel_left_wheel_link">
-    <inertial>
-      <origin xyz="0 0 0" rpy="0 0 0" />
-      <mass value="3.0" />
-      <inertia ixx="0.0091" ixy="0.0" ixz="0.0" iyy="0.0091" iyz="0.0" izz="0.015" />
-    </inertial>
-    <visual>
-      <origin xyz="0 0 0" rpy="1.5708 0 0" />
-      <geometry>
-        <cylinder radius="0.1" length="0.08" />
-      </geometry>
-      <material name="orange_wheel">
-        <color rgba="1.0 0.35 0.0 1.0" />
-      </material>
-    </visual>
-    <collision>
-      <origin xyz="0 0 0" rpy="1.5708 0 0" />
-      <geometry>
-        <cylinder radius="0.1" length="0.08" />
-      </geometry>
-    </collision>
-  </link>
-  <joint name="wheel_left_wheel_joint" type="revolute">
-    <parent link="wheel_left_steering_link" />
-    <child link="wheel_left_wheel_link" />
-    <origin xyz="0.0 0.0 0.0" rpy="0 0 0" />
-    <axis xyz="0 1 0" />
-    <limit lower="-1e9" upper="1e9" effort="10.0" velocity="10.0" />
-  </joint>
-  <!-- ==================== Right Steering Module ==================== -->
-  <link name="wheel_right_steering_link">
-    <inertial>
-      <origin xyz="0 0 0" rpy="0 0 0" />
-      <mass value="1.5" />
-      <inertia ixx="0.0045" ixy="0.0" ixz="0.0" iyy="0.0045" iyz="0.0" izz="0.0075" />
-    </inertial>
-    <visual>
-      <origin xyz="0 0 0" rpy="0 0 0" />
-      <geometry>
-        <cylinder radius="0.03" length="0.06" />
-      </geometry>
-      <material name="grey" />
-    </visual>
-  </link>
-  <joint name="wheel_right_steering_joint" type="revolute">
-    <parent link="base_link" />
-    <child link="wheel_right_steering_link" />
-    <origin xyz="-0.15 -0.20 -0.05" rpy="0 0 0" />
-    <axis xyz="0 0 1" />
-    <limit lower="-1.5708" upper="1.5708" effort="100.0" velocity="5.0" />
-  </joint>
-  <link name="wheel_right_wheel_link">
-    <inertial>
-      <origin xyz="0 0 0" rpy="0 0 0" />
-      <mass value="3.0" />
-      <inertia ixx="0.0091" ixy="0.0" ixz="0.0" iyy="0.0091" iyz="0.0" izz="0.015" />
-    </inertial>
-    <visual>
-      <origin xyz="0 0 0" rpy="1.5708 0 0" />
-      <geometry>
-        <cylinder radius="0.1" length="0.08" />
-      </geometry>
-      <material name="orange_wheel">
-        <color rgba="1.0 0.35 0.0 1.0" />
-      </material>
-    </visual>
-    <collision>
-      <origin xyz="0 0 0" rpy="1.5708 0 0" />
-      <geometry>
-        <cylinder radius="0.1" length="0.08" />
-      </geometry>
-    </collision>
-  </link>
-  <joint name="wheel_right_wheel_joint" type="revolute">
-    <parent link="wheel_right_steering_link" />
-    <child link="wheel_right_wheel_link" />
-    <origin xyz="0.0 0.0 0.0" rpy="0 0 0" />
-    <axis xyz="0 1 0" />
-    <limit lower="-1e9" upper="1e9" effort="10.0" velocity="10.0" />
-  </joint>
-  <!-- ==================== ros2_control ==================== -->
-  <ros2_control name="IgnitionSystem" type="system">
-    <hardware>
-      <plugin>ign_ros2_control/IgnitionSystem</plugin>
-    </hardware>
-    <joint name="wheel_front_steering_joint">
-      <command_interface name="position" />
-      <state_interface name="position" />
-      <state_interface name="velocity" />
-    </joint>
-    <joint name="wheel_left_steering_joint">
-      <command_interface name="position" />
-      <state_interface name="position" />
-      <state_interface name="velocity" />
-    </joint>
-    <joint name="wheel_right_steering_joint">
-      <command_interface name="position" />
-      <state_interface name="position" />
-      <state_interface name="velocity" />
-    </joint>
-    <joint name="wheel_front_wheel_joint">
-      <command_interface name="velocity" />
-      <state_interface name="position" />
-      <state_interface name="velocity" />
-    </joint>
-    <joint name="wheel_left_wheel_joint">
-      <command_interface name="velocity" />
-      <state_interface name="position" />
-      <state_interface name="velocity" />
-    </joint>
-    <joint name="wheel_right_wheel_joint">
-      <command_interface name="velocity" />
-      <state_interface name="position" />
-      <state_interface name="velocity" />
-    </joint>
-  </ros2_control>
-  <!-- ==================== Gazebo Plugins ==================== -->
-  <gazebo>
-    <plugin filename="ign_ros2_control-system" name="ign_ros2_control::IgnitionROS2ControlPlugin">
-      <parameters>$(find simulated_chassis)/param/three_wheel_controllers.yaml</parameters>
-      <robot_param>robot_description</robot_param>
-      <robot_param_node>robot_state_publisher</robot_param_node>
-    </plugin>
-    <plugin filename="ignition-gazebo-sensors-system" name="ignition::gazebo::systems::Sensors">
-    </plugin>
-    <plugin name="ignition::gazebo::systems::Imu" filename="ignition-gazebo-imu-system"></plugin>
-  </gazebo>
-  <!-- ==================== IMU Sensor ==================== -->
-  <gazebo reference="imu_link">
-    <sensor name="imu_sensor" type="imu">
-      <always_on>true</always_on>
-      <update_rate>100</update_rate>
-      <visualize>false</visualize>
-      <topic>/imu</topic>
-      <ignition_frame_id>imu_link</ignition_frame_id>
-      <imu>
-        <frame_id>imu_link</frame_id>
-        <!-- 角速度：白噪声密度约 0.01°/s/√Hz，
-           100Hz 下每采样 σ≈0.001 rad/s (0.057°/s)；
-           上电零偏 σ≈0.002°/s (3.5e-5 rad/s)；
-           零偏随机游走 10°/hr，相关时间 1000s -->
-        <angular_velocity>
-          <x>
-            <noise type="gaussian">
-              <mean>0.0</mean>
-              <stddev>0.001</stddev>
-              <bias_mean>0.0</bias_mean>
-              <bias_stddev>0.00005</bias_stddev>
-              <dynamic_bias_stddev>0.00005</dynamic_bias_stddev>
-              <dynamic_bias_correlation_time>1000.0</dynamic_bias_correlation_time>
-            </noise>
-          </x>
-          <y>
-            <noise type="gaussian">
-              <mean>0.0</mean>
-              <stddev>0.001</stddev>
-              <bias_mean>0.0</bias_mean>
-              <bias_stddev>0.00005</bias_stddev>
-              <dynamic_bias_stddev>0.00005</dynamic_bias_stddev>
-              <dynamic_bias_correlation_time>1000.0</dynamic_bias_correlation_time>
-            </noise>
-          </y>
-          <z>
-            <noise type="gaussian">
-              <mean>0.0</mean>
-              <stddev>0.001</stddev>
-              <bias_mean>0.0</bias_mean>
-              <bias_stddev>0.00005</bias_stddev>
-              <dynamic_bias_stddev>0.00005</dynamic_bias_stddev>
-              <dynamic_bias_correlation_time>1000.0</dynamic_bias_correlation_time>
-            </noise>
-          </z>
-        </angular_velocity>
-        <!-- 线加速度：白噪声密度约 60µg/√Hz，
-           100Hz 下每采样 σ≈0.0006 m/s²；
-           上电零偏 σ≈0.00015 m/s² (15µg)；
-           零偏随机游走 0.05mg，相关时间 1000s -->
-        <linear_acceleration>
-          <x>
-            <noise type="gaussian">
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