Commit message: 导航增加自由导航接口，tf局部代价地图，时间戳过期的bug解决方案，升级系统tf 安装包

File: src/simulated_chassis/urdf/three_wheel_chassis_2d.xacro (robot description, xacro)
@@ -50,6 +50,6 @@
         <box size="0.52 0.6 0.18" />
       </geometry>
-      <material name="green">
-        <color rgba="0.1 0.8 0.1 1.0" />
+      <material name="light_indigo">
+        <color rgba="0.471 0.549 0.871 1.0" />
       </material>
     </visual>
@@ -66,5 +66,5 @@
         <box size="0.14 0.46 0.18" />
       </geometry>
-      <material name="green" />
+      <material name="light_indigo" />
     </visual>
     <collision>
@@ -80,5 +80,5 @@
         <box size="0.14 0.46 0.18" />
       </geometry>
-      <material name="green" />
+      <material name="light_indigo" />
     </visual>
     <collision>
@@ -206,5 +206,5 @@
     <origin xyz="0.0 0.0 0.0" rpy="0 0 0" />
     <axis xyz="0 1 0" />
-    <limit lower="-1e9" upper="1e9" effort="10.0" velocity="10.0" />
+    <limit lower="-1e9" upper="1e9" effort="10.0" velocity="18.0" />
   </joint>
   <!-- ==================== Left Steering Module ==================== -->
@@ -257,5 +257,5 @@
     <origin xyz="0.0 0.0 0.0" rpy="0 0 0" />
     <axis xyz="0 1 0" />
-    <limit lower="-1e9" upper="1e9" effort="10.0" velocity="10.0" />
+    <limit lower="-1e9" upper="1e9" effort="10.0" velocity="18.0" />
   </joint>
   <!-- ==================== Right Steering Module ==================== -->
@@ -308,5 +308,5 @@
     <origin xyz="0.0 0.0 0.0" rpy="0 0 0" />
     <axis xyz="0 1 0" />
-    <limit lower="-1e9" upper="1e9" effort="10.0" velocity="10.0" />
+    <limit lower="-1e9" upper="1e9" effort="10.0" velocity="18.0" />
   </joint>
   <!-- ==================== ros2_control ==================== -->

File: src/simulated_chassis/urdf/three_wheel_chassis_3d_macro.xacro (robot description, xacro)
@@ -36,6 +36,6 @@
         <box size="0.8 0.6 0.18" />
       </geometry>
-      <material name="green">
-        <color rgba="0.1 0.8 0.1 1.0" />
+      <material name="light_indigo">
+        <color rgba="0.471 0.549 0.871 1.0" />
       </material>
     </visual>
@@ -206,5 +206,5 @@
     <origin xyz="0.0 0.0 0.0" rpy="0 0 0" />
     <axis xyz="0 1 0" />
-    <limit lower="-1e9" upper="1e9" effort="10.0" velocity="10.0" />
+    <limit lower="-1e9" upper="1e9" effort="10.0" velocity="18.0" />
   </joint>
   <!-- ==================== Left Steering Module ==================== -->
@@ -257,5 +257,5 @@
     <origin xyz="0.0 0.0 0.0" rpy="0 0 0" />
     <axis xyz="0 1 0" />
-    <limit lower="-1e9" upper="1e9" effort="10.0" velocity="10.0" />
+    <limit lower="-1e9" upper="1e9" effort="10.0" velocity="18.0" />
   </joint>
   <!-- ==================== Right Steering Module ==================== -->
@@ -308,5 +308,5 @@
     <origin xyz="0.0 0.0 0.0" rpy="0 0 0" />
     <axis xyz="0 1 0" />
-    <limit lower="-1e9" upper="1e9" effort="10.0" velocity="10.0" />
+    <limit lower="-1e9" upper="1e9" effort="10.0" velocity="18.0" />
   </joint>
   <!-- ==================== ros2_control ==================== -->
