Commit message: 解决了差速底盘移植到jazzy版本的ros2系统，无法正常运行的问题

File: src/jzt_robot/urdf/diff/common_properties.xacro (robot description, xacro)
@@ -8,20 +8,21 @@
     <xacro:property name="base_box_y" value="0.4" />
     <xacro:property name="base_box_z" value="0.12" />
-    <xacro:property name="base_mass" value="0.2" />
-    <xacro:property name="base_offset_z" value="0.005" />
-    <!-- 轮子参数 -->
-    <xacro:property name="wheel_radius" value="0.032" />
-    <xacro:property name="wheel_width" value="0.04" />
-    <xacro:property name="wheel_mass" value="0.2" />
-    <!-- 轮子位置 (相对于 base_link) -->
+    <xacro:property name="base_mass" value="50.0" />
+    <xacro:property name="base_offset_z" value="0.15" />
+    <!-- 轮子参数（直径18cm=半径9cm，可装电机转子） -->
+    <xacro:property name="wheel_radius" value="0.09" />
+    <xacro:property name="wheel_width" value="0.06" />
+    <xacro:property name="wheel_mass" value="0.5" />
+    <!-- 轮子位置 (相对于 base_link，轮心在底盘底部边缘) -->
     <xacro:property name="wheel_x" value="-0.02" />
     <xacro:property name="wheel_y" value="0.18" />
     <xacro:property name="wheel_z" value="-0.06" />
-    <!-- 差速插件运动学参数 -->
+    <!-- 差速运动学参数 -->
     <xacro:property name="wheel_separation" value="0.36" />
-    <xacro:property name="wheel_diameter" value="0.065" />
-    <!-- 脚轮参数 -->
-    <xacro:property name="caster_radius" value="0.016" />
-    <xacro:property name="caster_mass" value="0.02" />
+    <xacro:property name="wheel_diameter" value="0.18" />
+    <!-- 脚轮参数（比动力轮小，z略高于地面防止动力轮悬空） -->
+    <xacro:property name="caster_radius" value="0.03" />
+    <xacro:property name="caster_width" value="0.02" />
+    <xacro:property name="caster_mass" value="0.05" />
     <!-- 颜色定义 -->
     <material name="purple">

File: src/jzt_robot/urdf/diff/diff_wheels.xacro (robot description, xacro)
@@ -27,4 +27,12 @@
         <axis xyz="0 1 0" />
     </joint>
+    <!-- ==================== 左轮 ==================== -->
+    <!-- <joint name="left_wheel_joint" type="revolute">
+        <parent link="base_link" />
+        <child link="left_wheel_link" />
+        <origin xyz="${wheel_x} ${wheel_y} ${wheel_z}" />
+        <axis xyz="0 1 0" />
+        <limit lower="-1e9" upper="1e9" effort="100.0" velocity="100.0" />
+    </joint> -->
     <!-- ==================== 右轮 ==================== -->
     <link name="right_wheel_link">
@@ -53,11 +61,47 @@
         <axis xyz="0 1 0" />
     </joint>
-    <!-- ==================== 脚轮宏 ==================== -->
+    <!-- ==================== 右轮 ==================== -->
+    <!-- <joint name="right_wheel_joint" type="revolute">
+        <parent link="base_link" />
+        <child link="right_wheel_link" />
+        <origin xyz="${wheel_x} ${-wheel_y} ${wheel_z}" />
+        <axis xyz="0 1 0" />
+        <limit lower="-1e9" upper="1e9" effort="100.0" velocity="100.0" />
+    </joint> -->
+    <!-- ==================== 脚轮宏（圆柱形，黑色，含支架） ==================== -->
     <xacro:macro name="caster_wheel" params="prefix x y z">
+        <!-- 支架：连接底盘底部到万向轮 -->
+        <link name="${prefix}_bracket_link">
+            <visual>
+                <origin xyz="0 0 0" rpy="0 0 0" />
+                <geometry>
+                    <cylinder length="0.05" radius="0.012" />
+                </geometry>
+                <material name="dark_grey">
+                    <color rgba="0.3 0.3 0.3 1.0" />
+                </material>
+            </visual>
+            <collision>
+                <origin xyz="0 0 0" rpy="0 0 0" />
+                <geometry>
+                    <cylinder length="0.05" radius="0.012" />
+                </geometry>
+            </collision>
+            <inertial>
+                <mass value="0.05" />
+                <xacro:cylinder_inertia m="0.05" r="0.012" l="0.05" />
+            </inertial>
+        </link>
+        <joint name="${prefix}_bracket_joint" type="fixed">
+            <parent link="base_link" />
+            <child link="${prefix}_bracket_link" />
+            <origin xyz="${x} ${y} -0.085" />
+        </joint>
+        <!-- 万向轮 -->
         <link name="${prefix}_link">
             <visual>
                 <origin xyz="0 0 0" rpy="${PI_2} 0 0" />
                 <geometry>
-                    <sphere radius="${caster_radius}" />
+                    <cylinder length="${caster_width}" radius="${caster_radius}" />
                 </geometry>
                 <material name="black" />
@@ -66,10 +110,10 @@
                 <origin xyz="0 0 0" rpy="${PI_2} 0 0" />
                 <geometry>
-                    <sphere radius="${caster_radius}" />
+                    <cylinder length="${caster_width}" radius="${caster_radius}" />
                 </geometry>
             </collision>
             <inertial>
                 <mass value="${caster_mass}" />
-                <xacro:sphere_inertia m="${caster_mass}" r="${caster_radius}" />
+                <xacro:cylinder_inertia m="${caster_mass}" r="${caster_radius}" l="${caster_width}" />
             </inertial>
         </link>
@@ -81,7 +125,7 @@
     </xacro:macro>
     <!-- 四个脚轮 -->
-    <xacro:caster_wheel prefix="caster_front_right" x="0.28" y="0.18" z="-0.076" />
-    <xacro:caster_wheel prefix="caster_front_left"  x="0.28" y="-0.18" z="-0.076" />
-    <xacro:caster_wheel prefix="caster_rear_right"  x="-0.28" y="0.18" z="-0.076" />
-    <xacro:caster_wheel prefix="caster_rear_left"   x="-0.28" y="-0.18" z="-0.076" />
+    <xacro:caster_wheel prefix="caster_front_right" x="0.24" y="0.14" z="-0.115" />
+    <xacro:caster_wheel prefix="caster_front_left"  x="0.24" y="-0.14" z="-0.115" />
+    <xacro:caster_wheel prefix="caster_rear_right"  x="-0.24" y="0.14" z="-0.115" />
+    <xacro:caster_wheel prefix="caster_rear_left"   x="-0.24" y="-0.14" z="-0.115" />
 </robot>

File: src/jzt_robot/urdf/diff/sensors_gazebo.xacro (robot description, xacro)
@@ -3,8 +3,10 @@
     <!-- ==================== 前向激光雷达 (270°) ==================== -->
     <gazebo reference="laser_front_link">
-        <sensor name="laser_front_sensor" type="ray">
+        <sensor name="laser_front_sensor" type="gpu_ray">
             <always_on>true</always_on>
             <update_rate>20</update_rate>
             <visualize>true</visualize>
+            <topic>/model/jzDiffRobot/laser_front_link/scan</topic>
+            <gz_frame_id>laser_front_link</gz_frame_id>
             <pose>0 0 0 0 0 0</pose>
             <ray>
@@ -32,8 +34,10 @@
     <!-- ==================== 后向激光雷达 (270°) ==================== -->
     <gazebo reference="laser_rear_link">
-        <sensor name="laser_rear_sensor" type="ray">
+        <sensor name="laser_rear_sensor" type="gpu_ray">
             <always_on>true</always_on>
             <update_rate>20</update_rate>
             <visualize>true</visualize>
+            <topic>/model/jzDiffRobot/laser_rear_link/scan</topic>
+            <gz_frame_id>laser_rear_link</gz_frame_id>
             <pose>0 0 0 0 0 0</pose>
             <ray>
@@ -113,3 +117,2 @@
     </gazebo>
 </robot>
-</robot>
