Commit message: 仿真机器人bug修复，实现了jazzy平台的仿真，建图，离线建图，导航的各种功能

File: src/jzt_robot/urdf/diff/robot.xacro (robot description, xacro)
@@ -1,4 +1,4 @@
 <?xml version="1.0"?>
-<robot name="jzDiffRobot"
+<robot name="$(arg robot_name)"
     xmlns:xacro="http://ros.org/wiki/xacro">
     <!--
@@ -6,4 +6,7 @@
     传感器：前270° 激光 + 后270° 激光 + IMU
     -->
+    <xacro:arg name="robot_name" default="jzDiffRobot"/>
+    <!-- 转为 property 供子文件使用 -->
+    <xacro:property name="robot_name" value="$(arg robot_name)"/>
     <!-- 载入核心结构（常量、底盘、轮子） -->
     <xacro:include filename="common_properties.xacro" />

File: src/jzt_robot/urdf/diff/sensors_gazebo.xacro (robot description, xacro)
@@ -7,5 +7,5 @@
             <update_rate>20</update_rate>
             <visualize>true</visualize>
-            <topic>/model/jzDiffRobot/laser_front_link/scan</topic>
+            <topic>/model/${robot_name}/laser_front_link/scan</topic>
             <gz_frame_id>laser_front_link</gz_frame_id>
             <pose>0 0 0 0 0 0</pose>
@@ -38,5 +38,5 @@
             <update_rate>20</update_rate>
             <visualize>true</visualize>
-            <topic>/model/jzDiffRobot/laser_rear_link/scan</topic>
+            <topic>/model/${robot_name}/laser_rear_link/scan</topic>
             <gz_frame_id>laser_rear_link</gz_frame_id>
             <pose>0 0 0 0 0 0</pose>
