Commit message: update before switch branch

File: src/zioneer_robot/urdf/diff/common_properties.xacro (robot description, xacro)
@@ -21,6 +21,6 @@
     <xacro:property name="wheel_separation" value="0.36" />
     <xacro:property name="wheel_diameter" value="0.18" />
-    <!-- 脚轮参数（比动力轮小，z略高于地面防止动力轮悬空） -->
-    <xacro:property name="caster_radius" value="0.03" />
+    <!-- 脚轮参数（比动力轮小，轮底略高于地面，确保驱动轮接地有牵引力） -->
+    <xacro:property name="caster_radius" value="0.028" />
     <xacro:property name="caster_width" value="0.02" />
     <xacro:property name="caster_mass" value="0.05" />

File: src/zioneer_robot/urdf/diff/diff_wheels.xacro (robot description, xacro)
@@ -108,5 +108,5 @@
         </joint>
     </xacro:macro>
-    <!-- 四个脚轮：z=-0.1205，底部低于地面0.5mm预紧，防止机器人两点支撑翘起1.1° -->
+    <!-- 四个脚轮：z=-0.1205，半径0.028，轮底高于地面1.5mm，驱动轮接地 -->
     <xacro:caster_wheel prefix="caster_front_right" x="0.24" y="0.14" z="-0.1205" />
     <xacro:caster_wheel prefix="caster_front_left"  x="0.24" y="-0.14" z="-0.1205" />
