Commit message: 上位机 URDF/mesh 链路打通(U1/U2):params_glob 裸参数名 + 共享 mesh 服务 + 双描述
- U1(真根因修复):rosapi params_glob 匹配的是裸参数名(无节点前缀),
  '/robot_state_publisher/*' 匹配不到 robot_description;三处白名单补
  'robot_description' 精确项
- U2:mesh 静态服务挪到 agv_bridge_v2 共享,simulated_chassis_ur5e bridge
  同样默认拉起(8090);实测命中系统包 ur_description 的 .dae(358KB/200)
- U2.5(新发现并修复):组合 URDF 因 sim_ignition=true 被官方宏展开成
  file:// 绝对路径 mesh,前端只重写 package:// 导致永远加载不了;
  改为双描述——Gazebo 拉起用 file:// 版(零风险不变),robot_state_publisher
  用 package:// 版(14 处 mesh 全部可经 8090 拉取)
  (three_wheel_sim 新增 rsp_description_file 参数,缺省同 description_file,
  纯底盘行为不变)
- U3 复核:本地 RSP+伪关节态验证 steering/wheel link TF 均正常发布,
  判定为测试环境代码未更新,无需改代码

File: src/simulated_chassis_ur5e/urdf/arm_mount.xacro (robot description, xacro)
@@ -2,5 +2,5 @@
 <robot xmlns:xacro="http://www.ros.org/wiki/xacro">
   <xacro:include filename="$(find ur_description)/urdf/ur_macro.xacro"/>
-  <xacro:macro name="mounted_ur5e" params="mounting_file">
+  <xacro:macro name="mounted_ur5e" params="mounting_file sim_ignition:=true">
     <xacro:property name="mount" value="${xacro.load_yaml(mounting_file)}"/>
     <xacro:property name="h" value="${mount['pedestal_height']}"/>
@@ -20,4 +20,6 @@
       <origin xyz="${mount['xyz']}" rpy="${mount['rpy']}"/>
     </joint>
+    <!-- sim_ignition=true 时官方宏把 mesh 写成 file:// 绝对路径(Gazebo 解析需要);
+         false 时保持 package://(上位机前端按 VITE_URDF_MESH_BASE 重写拉取 mesh) -->
     <xacro:ur_robot name="UR5eSystem" tf_prefix="ur5e_" parent="arm_mount_link" ur_type="ur5e"
       joint_limits_parameters_file="$(find ur_description)/config/ur5e/joint_limits.yaml"
@@ -25,5 +27,5 @@
       physical_parameters_file="$(find ur_description)/config/ur5e/physical_parameters.yaml"
       visual_parameters_file="$(find ur_description)/config/ur5e/visual_parameters.yaml"
-      sim_ignition="true" safety_limits="true"
+      sim_ignition="${sim_ignition}" safety_limits="true"
       initial_positions="${xacro.load_yaml('$(find simulated_ur5e)/config/initial_positions.yaml')}">
       <origin xyz="0 0 ${h}" rpy="0 0 0"/>

File: src/simulated_chassis_ur5e/urdf/robot.urdf.xacro (robot description, xacro)
@@ -3,7 +3,9 @@
   <xacro:arg name="controllers_file" default="$(find simulated_chassis_ur5e)/config/controllers.yaml"/>
   <xacro:arg name="mounting_file" default="$(find simulated_chassis_ur5e)/config/mounting.yaml"/>
+  <!-- sim_ignition=true: mesh 用 file:// 绝对路径(Gazebo);false: package://(上位机) -->
+  <xacro:arg name="sim_ignition" default="true"/>
   <xacro:include filename="$(find simulated_chassis)/urdf/three_wheel_chassis_3d_macro.xacro"/>
   <xacro:include filename="$(find simulated_chassis_ur5e)/urdf/arm_mount.xacro"/>
   <xacro:three_wheel_chassis_3d controllers_file="$(arg controllers_file)" lidar_collisions="true"/>
-  <xacro:mounted_ur5e mounting_file="$(arg mounting_file)"/>
+  <xacro:mounted_ur5e mounting_file="$(arg mounting_file)" sim_ignition="$(arg sim_ignition)"/>
 </robot>
