Commit message: 1：修复任务执行失败，返回错误信息含糊的问题，2：增加导航执行任务的超时时长，3：增加夹爪末端

File: src/simulated_chassis_ur5e/config/moveit/robot.srdf.xacro (robot description, xacro)
@@ -3,4 +3,21 @@
   <xacro:include filename="$(find ur_moveit_config)/srdf/ur_macro.srdf.xacro"/>
   <xacro:ur_srdf name="ur" prefix="ur5e_"/>
+  <xacro:arg name="tool_type" default="gripper"/>
+  <xacro:arg name="gripper_file" default="$(find simulated_chassis_ur5e)/config/gripper.yaml"/>
+  <xacro:if value="${'$(arg tool_type)' == 'gripper'}">
+    <xacro:property name="grip" value="${xacro.load_yaml('$(arg gripper_file)')}"/>
+    <group name="ur5e_gripper"><joint name="ur5e_gripper_left_joint"/><joint name="ur5e_gripper_right_joint"/></group>
+    <group_state name="open" group="ur5e_gripper">
+      <joint name="ur5e_gripper_left_joint" value="${grip['max_width']/2}"/><joint name="ur5e_gripper_right_joint" value="${grip['max_width']/2}"/>
+    </group_state>
+    <group_state name="closed" group="ur5e_gripper">
+      <joint name="ur5e_gripper_left_joint" value="0"/><joint name="ur5e_gripper_right_joint" value="0"/>
+    </group_state>
+    <end_effector name="parallel_gripper" parent_link="ur5e_gripper_tcp" group="ur5e_gripper" parent_group="ur5e_ur_manipulator"/>
+    <disable_collisions link1="ur5e_wrist_3_link" link2="ur5e_gripper_base" reason="Adjacent"/>
+    <disable_collisions link1="ur5e_gripper_base" link2="ur5e_gripper_left_finger" reason="Adjacent"/>
+    <disable_collisions link1="ur5e_gripper_base" link2="ur5e_gripper_right_finger" reason="Adjacent"/>
+    <disable_collisions link1="ur5e_gripper_left_finger" link2="ur5e_gripper_right_finger" reason="Touching"/>
+  </xacro:if>
   <xacro:property name="initial" value="${xacro.load_yaml('$(find simulated_ur5e)/config/initial_positions.yaml')}"/>
   <group_state name="stowed" group="ur5e_ur_manipulator">

File: src/simulated_chassis_ur5e/urdf/robot.urdf.xacro (robot description, xacro)
@@ -6,4 +6,7 @@
   <xacro:arg name="sim_ignition" default="true"/>
   <xacro:arg name="camera_file" default="$(find simulated_chassis_ur5e)/config/wrist_camera.yaml"/>
+  <xacro:arg name="tool_type" default="gripper"/>
+  <xacro:arg name="gripper_file" default="$(find simulated_chassis_ur5e)/config/gripper.yaml"/>
+  <xacro:include filename="$(find simulated_chassis_ur5e)/urdf/gripper.xacro"/>
   <xacro:include filename="$(find simulated_chassis_ur5e)/urdf/wrist_camera.xacro"/>
   <xacro:include filename="$(find simulated_chassis)/urdf/three_wheel_chassis_3d_macro.xacro"/>
@@ -11,4 +14,5 @@
   <xacro:three_wheel_chassis_3d controllers_file="$(arg controllers_file)" lidar_collisions="true"/>
   <xacro:mounted_ur5e mounting_file="$(arg mounting_file)" sim_ignition="$(arg sim_ignition)"/>
-  <xacro:wrist_camera camera_file="$(arg camera_file)"/>
+  <xacro:if value="${'$(arg tool_type)' == 'camera'}"><xacro:wrist_camera camera_file="$(arg camera_file)"/></xacro:if>
+  <xacro:if value="${'$(arg tool_type)' == 'gripper'}"><xacro:parallel_gripper gripper_file="$(arg gripper_file)"/></xacro:if>
 </robot>
